File: Schematic/STM32_USB_ECG_B2_InstAmp.kicad_sch (KiCad schematic)
At the start: 135 parts, among them J101 ECG Cable, U101 TL074, U102 TL074, U103 TL074, U104 CD4066, U105 CD4066, U106 AD823ANZ, U107 TL431DBZ, U108 74HC4051, U109 TL072

Commit message: Update new fixed schematic
Connections:
- net VREF: now also C110.2
Other:
- moved on the sheet: C101, C102, C103, C104, C105, C106, C107, C108, C109, C110, C111, C112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
