File: Schematic/STM32_USB_ECG_B3_ADC_MCU_PSU.kicad_sch (KiCad schematic)
At the start: 92 parts, among them J201 AVR-ISP-6, J202 USB_B, Q201 MMBT3906, Q202 2SK3225, Q203 2SK3225, T201 Pulse Xfmr, U201 MCP3202BI/P, U202 MCP4725xxx-xCH, U203 ICL7660, U204 ATmega328P-AU, U205 LM78M05_TO252, U206 LM78M05_TO252, U207 6N137, U208 6N137, U209 74HC04, U210 UCC27324, U211 AMS1117-3.3, U212 STM32F401CCUx, Y201 16 MHz, Y202 25 MHz

Commit message: Update new fixed schematic
Other:
- moved on the sheet: C201, C202, C203, C204, C205, C206, C207, C208, C209, C210, C211, C212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
